File: KiCad/coincall/coincall.kicad_pcb (KiCad board)
At the start: 2 copper layers, 40.6 x 27.9 mm, 3 parts

Commit message: Nov 23th
Parts:
- removed BT1: 3.7V, Battery:BatteryHolder_Keystone_1058_1x2032
- removed D1: RED, Diode_SMD:D_0603_1608Metric
- removed R1: 1K, Resistor_SMD:R_0603_1608Metric
- added BT4: 3V, Battery:BatteryHolder_Keystone_1057_1x2032, B.Cu at (178.8, 99.1)
- added D4: RED, Diode_SMD:D_0603_1608Metric, F.Cu at (193.0, 113.0)
- added R4: 1K, Resistor_SMD:R_0603_1608Metric, F.Cu at (164.0, 113.0)
Routing:
- net Net-(D4-A): track 0.00 -> 27.4 mm
- net Net-(D1-A): track 25.5 -> 0.00 mm
- net +5V: track 0.00 -> 14.2 mm, vias 0 -> 1
- net VCC: track 10.6 -> 0.00 mm, vias 1 -> 0
- net GND: track 10.5 -> 14.1 mm
- added copper zone on F.Cu, net GND
Other:
- board size 40.6 x 27.9 mm -> 41 x 32 mm
