File: KiCad/coincall/coincall.kicad_sch (KiCad schematic)
At the start: 3 parts

Commit message: Nov 23th
Parts:
- added D5, D6: LED, symbol Device:LED
- added R5, R6: 1K, Resistor_SMD:R_0603_1608Metric, symbol Device:R_US
- BT4: renamed from BT1; value 3.7V -> 3V; footprint Battery:BatteryHolder_Keystone_1058_1x2032 -> Battery:BatteryHolder_Keystone_1057_1x2032
- renumbered D1 to D4, R1 to R4
Connections:
- net GND: now also BT4.2 (-), D4.1 (K), D5.1 (K), D6.1 (K)
- net +5V: now reaches R4.1
- net +5V: now also BT4.1 (+), R5.1
- net at R4.2: now also D4.2 (A)
- new net: D6.2 (A), R6.2
- new net: D5.2 (A), R5.2
- new net +3V3: R6.1
