File: KiCad/arduino_robotarm_shield/arduino_robotarm_shield.kicad_pcb (KiCad board)
At the start: 2 copper layers, 57.1 x 53.4 mm, 10 parts, among them J1 Screw_Terminal_01x02, J2 Conn_01x03, J3 Conn_01x03, J4 Conn_01x03, J5 Conn_01x03, J6 Conn_01x03, J7 Conn_01x03

Commit message: Nov 23th
Parts:
- moved D1 43.7 mm to (165.5, 66.0)
- moved R1 42.8 mm to (154.5, 66.0), turned to 180 degrees
- moved A1 16.2 mm to (143.6, 81.1)
- moved J1 10.9 mm to (132.7, 58.3)
- moved J7 9.60 mm to (147.0, 43.5)
- moved J6 9.16 mm to (152.0, 43.5)
- moved J5 8.73 mm to (157.0, 43.5)
- moved J4 8.31 mm to (162.0, 43.5)
- moved J3 7.92 mm to (167.0, 43.5)
- moved J2 7.51 mm to (172.0, 43.5)
Routing:
- net GND: track 127.2 -> 100.3 mm
- net /S3: track 25.9 -> 11.1 mm
- net /S4: track 25.1 -> 10.6 mm
- net -5V: track 57.0 -> 71.5 mm
- net /S1: track 25.0 -> 10.6 mm
- net /S0: track 24.6 -> 10.5 mm
- net /S2: track 24.0 -> 11.2 mm
- net /S5: track 24.3 -> 12.1 mm
- net Net-(D1-K): track 7.59 -> 11.0 mm
- added copper zone on B.Cu, net GND
Other:
- outline, holes or cut-outs redrawn

Commit message: Dec25th
Parts:
- added J8: Conn_01x04, Connector_PinHeader_2.54mm:PinHeader_1x04_P2.54mm_Vertical, F.Cu at (177.5, 65.8)
Connections:
- A1 pad 13: unconnected-(A1-SDA/A4-Pad13) -> /SDA
- A1 pad 14: unconnected-(A1-SCL/A5-Pad14) -> /SCL
Routing:
- net GND: track 100.3 -> 124.3 mm
- net /SDA: track 0.00 -> 18.5 mm
- net /SCL: track 0.00 -> 17.4 mm
- net -5V: track 71.5 -> 84.5 mm
Changed lines of the file:
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@@
   (net 10 "unconnected-(A1-A2-Pad11)")
   (net 11 "unconnected-(A1-A3-Pad12)")
-  (net 12 "unconnected-(A1-SDA{slash}A4-Pad13)")
-  (net 13 "unconnected-(A1-SCL{slash}A5-Pad14)")
+  (net 12 "/SDA")
+  (net 13 "/SCL")
   (net 14 "unconnected-(A1-D0{slash}RX-Pad15)")
   (net 15 "unconnected-(A1-D1{slash}TX-Pad16)")
@@
     )
   )
+  (footprint "Connector_PinHeader_2.54mm:PinHeader_1x04_P2.54mm_Vertical" (layer "F.Cu")
+    (at 177.546 65.786)
+    (descr "Through hole straight pin header, 1x04, 2.54mm pitch, single row")
+    (tags "Through hole pin header THT 1x04 2.54mm single row")
+    (property "Sheetfile" "arduino_robotarm_shield.kicad_sch")
+    (property "Sheetname" "")
+    (property "ki_description" "Generic connector, single row, 01x04, script generated (kicad-library-utils/schlib/autogen/connector/)")
+    (property "ki_keywords" "connector")
+    (attr through_hole)
+    (fp_text reference "J8" (at 0 -2.33) (layer "F.SilkS")
+        (effects (font (size 1 1) (thickness 0.15)))
+    )
+    (fp_text value "Conn_01x04" (at 0 9.95) (layer "F.Fab")
+        (effects (font (size 1 1) (thickness 0.15)))
+    )
+    (fp_text user "${REFERENCE}" (at 0 3.81 90) (layer "F.Fab")
+        (effects (font (size 1 1) (thickness 0.15)))
+    )
+    (fp_line (start -1.33 -1.33) (end 0 -1.33)
+      (stroke (width 0.12) (type solid)) (layer "F.SilkS"))
+    (fp_line (start -1.33 0) (end -1.33 -1.33)
+      (stroke (width 0.12) (type solid)) (layer "F.SilkS"))
+    (fp_line (start -1.33 1.27) (end -1.33 8.95)
+      (stroke (width 0.12) (type solid)) (layer "F.SilkS"))
+    (fp_line (start -1.33 1.27) (end 1.33 1.27)
+      (stroke (width 0.12) (type solid)) (layer "F.SilkS"))
+    (fp_line (start -1.33 8.95) (end 1.33 8.95)
+      (stroke (width 0.12) (type solid)) (layer "F.SilkS"))
+    (fp_line (start 1.33 1.27) (end 1.33 8.95)
+      (stroke (width 0.12) (type solid)) (layer "F.SilkS"))
+    (fp_line (start -1.8 -1.8) (end -1.8 9.4)
+      (stroke (width 0.05) (type solid)) (layer "F.CrtYd"))
+    (fp_line (start -1.8 9.4) (end 1.8 9.4)
+      (stroke (width 0.05) (type solid)) (layer "F.CrtYd"))
+    (fp_line (start 1.8 -1.8) (end -1.8 -1.8)
+      (stroke (width 0.05) (type solid)) (layer "F.CrtYd"))
+    (fp_line (start 1.8 9.4) (end 1.8 -1.8)
+      (stroke (width 0.05) (type solid)) (layer "F.CrtYd"))
+    (fp_line (start -1.27 -0.635) (end -0.635 -1.27)
+      (stroke (width 0.1) (type solid)) (layer "F.Fab"))
+    (fp_line (start -1.27 8.89) (end -1.27 -0.635)
+      (stroke (width 0.1) (type solid)) (layer "F.Fab"))
+    (fp_line (start -0.635 -1.27) (end 1.27 -1.27)
+      (stroke (width 0.1) (type solid)) (layer "F.Fab"))
+    (fp_line (start 1.27 -1.27) (end 1.27 8.89)
+      (stroke (width 0.1) (type solid)) (layer "F.Fab"))
+    (fp_line (start 1.27 8.89) (end -1.27 8.89)
+      (stroke (width 0.1) (type solid)) (layer "F.Fab"))
+    (pad "1" thru_hole rect (at 0 0) (size 1.7 1.7) (drill 1) (layers "*.Cu" "*.Mask")
+      (net 12 "/SDA") (pinfunction "Pin_1") (pintype "passive"))
+    (pad "2" thru_hole oval (at 0 2.54) (size 1.7 1.7) (drill 1) (layers "*.Cu" "*.Mask")
+      (net 13 "/SCL") (pinfunction "Pin_2") (pintype "passive"))
+    (pad "3" thru_hole oval (at 0 5.08) (size 1.7 1.7) (drill 1) (layers "*.Cu" "*.Mask")
+      (net 26 "-5V") (pinfunction "Pin_3") (pintype "passive"))
+    (pad "4" thru_hole oval (at 0 7.62) (size 1.7 1.7) (drill 1) (layers "*.Cu" "*.Mask")
+      (net 6 "GND") (pinfunction "Pin_4") (pintype "passive"))
+    (model "${KICAD6_3DMODEL_DIR}/Connector_PinHeader_2.54mm.3dshapes/PinHeader_1x04_P2.54mm_Vertical.wrl"
+      (offset (xyz 0 0 0))
+      (scale (xyz 1 1 1))
+      (rotate (xyz 0 0 0))
+    )
+  )
   (footprint "LED_THT:LED_D5.0mm" (layer "F.Cu")
     (at 165.46 66)
@@
       (net 11 "unconnected-(A1-A3-Pad12)") (pinfunction "A3") (pintype "bidirectional+no_connect"))
     (pad "13" thru_hole oval (at 33.02 0 270) (size 1.6 1.6) (drill 1) (layers "*.Cu" "*.Mask")
-      (net 12 "unconnected-(A1-SDA{slash}A4-Pad13)") (pinfunction "SDA/A4") (pintype "bidirectional+no_connect"))
+      (net 12 "/SDA") (pinfunction "SDA/A4") (pintype "bidirectional"))
     (pad "14" thru_hole oval (at 35.56 0 270) (size 1.6 1.6) (drill 1) (layers "*.Cu" "*.Mask")
-      (net 13 "unconnected-(A1-SCL{slash}A5-Pad14)") (pinfunction "SCL/A5") (pintype "bidirectional+no_connect"))
+      (net 13 "/SCL") (pinfunction "SCL/A5") (pintype "bidirectional"))
     (pad "15" thru_hole oval (at 35.56 -48.26 270) (size 1.6 1.6) (drill 1) (layers "*.Cu" "*.Mask")
       (net 14 "unconnected-(A1-D0{slash}RX-Pad15)") (pinfunction "D0/RX") (pintype "bidirectional+no_connect"))
@@
   (segment (start 152.025 48.555) (end 157.025 48.555) (width 0.25) (layer "F.Cu") (net 6))
   (segment (start 149.5 66) (end 135.39 66) (width 0.25) (layer "F.Cu") (net 6))
+  (segment (start 161.544 74.676) (end 161.544 78.921229) (width 0.25) (layer "B.Cu") (net 6))
+  (segment (start 159.38668 81.078549) (end 159.266469 81.078549) (width 0.25) (layer "B.Cu") (net 6))
+  (segment (start 177.546 73.406) (end 162.814 73.406) (width 0.25) (layer "B.Cu") (net 6))
+  (segment (start 161.544 78.921229) (end 159.38668 81.078549) (width 0.25) (layer "B.Cu") (net 6))
+  (segment (start 162.814 73.406) (end 161.544 74.676) (width 0.25) (layer "B.Cu") (net 6))
+  (segment (start 176.767661 81.12) (end 176.66 81.12) (width 0.25) (layer "F.Cu") (net 12))
+  (segment (start 175.768 65.786) (end 174.244 67.31) (width 0.25) (layer "F.Cu") (net 12))
+  (segment (start 176.66 80.14) (end 176.66 80.74444) (width 0.25) (layer "F.Cu") (net 12))
+  (segment (start 174.244 77.724) (end 176.66 80.14) (width 0.25) (layer "F.Cu") (net 12))
+  (segment (start 177.546 65.786) (end 175.768 65.786) (width 0.25) (layer "F.Cu") (net 12))
+  (segment (start 174.244 67.31) (end 174.244 77.724) (width 0.25) (layer "F.Cu") (net 12))
+  (segment (start 176.782814 81.104847) (end 176.767661 81.12) (width 0.25) (layer "F.Cu") (net 12))
+  (segment (start 179.124104 81.50756) (end 179.358047 81.50756) (width 0.25) (layer "F.Cu") (net 13))
+  (segment (start 179.586469 81.279138) (end 179.586469 81.078549) (width 0.25) (layer "F.Cu") (net 13))
+  (segment (start 175.768 68.326) (end 175.514 68.58) (width 0.25) (layer "F.Cu") (net 13))
+  (segment (start 179.358047 81.50756) (end 179.586469 81.279138) (width 0.25) (layer "F.Cu") (net 13))
+  (segment (start 178.983863 81.44947) (end 179.124104 81.50756) (width 0.25) (layer "F.Cu") (net 13))
+  (segment (start 175.514 68.58) (end 175.514 77.979607) (width 0.25) (layer "F.Cu") (net 13))
+  (segment (start 175.514 77.979607) (end 178.983863 81.44947) (width 0.25) (layer "F.Cu") (net 13))
+  (segment (start 177.546 68.326) (end 175.768 68.326) (width 0.25) (layer "F.Cu") (net 13))
   (segment (start 165.46 66) (end 154.5 66) (width 0.25) (layer "F.Cu") (net 25))
   (segment (start 173 64) (end 170 64) (width 0.25) (layer "F.Cu") (net 26))
@@
   (segment (start 152.025 46.015) (end 157.025 46.015) (width 0.25) (layer "F.Cu") (net 26))
   (segment (start 174 46) (end 175 47) (width 0.25) (layer "F.Cu") (net 26))
+  (segment (start 168 66) (end 168 68.432) (width 0.25) (layer "B.Cu") (net 26))
   (segment (start 132.695 58.305) (end 134.735 58.305) (width 0.25) (layer "B.Cu") (net 26))
+  (segment (start 172.974 69.85) (end 173.99 70.866) (width 0.25) (layer "B.Cu") (net 26))
+  (segment (start 169.418 69.85) (end 172.974 69.85) (width 0.25) (layer "B.Cu") (net 26))
+  (segment (start 173.99 70.866) (end 177.546 70.866) (width 0.25) (layer "B.Cu") (net 26))
   (segment (start 134.735 58.305) (end 147.025 46.015) (width 0.25) (layer "B.Cu") (net 26))
+  (segment (start 168 68.432) (end 169.418 69.85) (width 0.25) (layer "B.Cu") (net 26))
   (segment (start 172 32.96208) (end 171.986469 32.948549) (width 0.25) (layer "F.Cu") (net 27))
   (segment (start 172 43.46) (end 172 32.96208) (width 0.25) (layer "F.Cu") (net 27))
@@
   (segment (start 147.307274 35.864333) (end 150.152469 33.019138) (width 0.25) (layer "F.Cu") (net 32))
   (segment (start 147.025 35.864333) (end 147.307274 35.864333) (width 0.25) (layer "F.Cu") (net 32))
-  (zone (net 6) (net_name "GND") (layers "F&B.Cu") (hatch edge 0.5)
+  (zone (net 6) (net_name "GND") (layer "F.Cu") (hatch edge 0.5)
     (connect_pads (clearance 0.5))
     (min_thickness 0.25) (filled_areas_thickness no)
@@
     (polygon
       (pts
-        (xy 107 28)
-        (xy 186 28)
-        (xy 186 86)
-        (xy 107 86)
+        (xy 108 29)
+        (xy 185 29)
+        (xy 185 85)
+        (xy 108 85)
       )
     )
+  )
+  (zone (net 6) (net_name "GND") (layer "B.Cu") (hatch edge 0.5)
+    (priority 1)
+    (connect_pads (clearance 0.5))
+    (min_thickness 0.25) (filled_areas_thickness no)
+    (fill yes (thermal_gap 0.5) (thermal_bridge_width 0.5))
+    (polygon
+      (pts
+        (xy 108 29)
+        (xy 185 29)
+        (xy 185 85)
+        (xy 108 85)
+      )
+    )
