File: KiCad/arduino_robotarm_shield/arduino_robotarm_shield.kicad_sch (KiCad schematic)
At the start: 10 parts, among them J1 Screw_Terminal_01x02, J2 Conn_01x03, J3 Conn_01x03, J4 Conn_01x03, J5 Conn_01x03, J6 Conn_01x03, J7 Conn_01x03

Commit message: Nov 23th
Changed lines of the file:
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@@
 (kicad_sch (version 20230121) (generator eeschema)
   (paper "A4")
-  (junction (at 158.75 105.41) (diameter 0) (color 0 0 0 0)
-  )
-  (junction (at 189.23 90.17) (diameter 0) (color 0 0 0 0)
-  )
-  (junction (at 111.76 125.73) (diameter 0) (color 0 0 0 0)
-  )
-  (junction (at 162.56 102.87) (diameter 0) (color 0 0 0 0)
-  )
-  (junction (at 189.23 102.87) (diameter 0) (color 0 0 0 0)
-  )
-  (junction (at 186.69 118.11) (diameter 0) (color 0 0 0 0)
-  )
-  (junction (at 186.69 105.41) (diameter 0) (color 0 0 0 0)
-  )
-  (junction (at 158.75 118.11) (diameter 0) (color 0 0 0 0)
-  )
-  (junction (at 162.56 90.17) (diameter 0) (color 0 0 0 0)
-  )
-  (bus (pts (xy 154.94 113.03) (xy 166.37 113.03))
-    (stroke (width 0) (type default))
-  )
-  (bus (pts (xy 186.69 92.71) (xy 186.69 105.41))
-    (stroke (width 0) (type default))
-  )
-  (bus (pts (xy 189.23 102.87) (xy 189.23 90.17))
-    (stroke (width 0) (type default))
-  )
-  (bus (pts (xy 152.4 73.66) (xy 148.59 73.66))
-    (stroke (width 0) (type default))
-  )
-  (bus (pts (xy 114.3 120.65) (xy 114.3 125.73))
-    (stroke (width 0) (type default))
-  )
-  (bus (pts (xy 193.04 102.87) (xy 189.23 102.87))
-    (stroke (width 0) (type default))
-  )
-  (bus (pts (xy 158.75 118.11) (xy 158.75 121.92))
-    (stroke (width 0) (type default))
-  )
-  (bus (pts (xy 186.69 105.41) (xy 193.04 105.41))
-    (stroke (width 0) (type default))
-  )
-  (bus (pts (xy 148.59 66.04) (xy 148.59 71.12))
-    (stroke (width 0) (type default))
-  )
-  (bus (pts (xy 186.69 105.41) (xy 186.69 118.11))
-    (stroke (width 0) (type default))
-  )
-  (bus (pts (xy 88.9 92.71) (xy 99.06 92.71))
-    (stroke (width 0) (type default))
-  )
-  (bus (pts (xy 148.59 71.12) (xy 152.4 71.12))
-    (stroke (width 0) (type default))
-  )
-  (bus (pts (xy 158.75 92.71) (xy 158.75 105.41))
-    (stroke (width 0) (type default))
-  )
-  (bus (pts (xy 138.43 72.39) (xy 138.43 81.28))
-    (stroke (width 0) (type default))
-  )
-  (bus (pts (xy 166.37 115.57) (xy 162.56 115.57))
-    (stroke (width 0) (type default))
-  )
-  (bus (pts (xy 189.23 83.82) (xy 189.23 90.17))
-    (stroke (width 0) (type default))
-  )
-  (bus (pts (xy 88.9 90.17) (xy 99.06 90.17))
-    (stroke (width 0) (type default))
-  )
-  (bus (pts (xy 182.88 100.33) (xy 193.04 100.33))
-    (stroke (width 0) (type default))
-  )
-  (bus (pts (xy 158.75 105.41) (xy 166.37 105.41))
-    (stroke (width 0) (type default))
-  )
-  (bus (pts (xy 138.43 88.9) (xy 138.43 95.25))
-    (stroke (width 0) (type default))
-  )
-  (bus (pts (xy 166.37 102.87) (xy 162.56 102.87))
-    (stroke (width 0) (type default))
-  )
-  (bus (pts (xy 88.9 85.09) (xy 99.06 85.09))
-    (stroke (width 0) (type default))
-  )
-  (bus (pts (xy 154.94 100.33) (xy 166.37 100.33))
-    (stroke (width 0) (type default))
-  )
-  (bus (pts (xy 166.37 90.17) (xy 162.56 90.17))
-    (stroke (width 0) (type default))
-  )
-  (bus (pts (xy 88.9 102.87) (xy 99.06 102.87))
-    (stroke (width 0) (type default))
-  )
-  (bus (pts (xy 193.04 118.11) (xy 186.69 118.11))
-    (stroke (width 0) (type default))
-  )
-  (bus (pts (xy 189.23 115.57) (xy 189.23 102.87))
-    (stroke (width 0) (type default))
-  )
-  (bus (pts (xy 114.3 125.73) (xy 111.76 125.73))
-    (stroke (width 0) (type default))
-  )
-  (bus (pts (xy 186.69 118.11) (xy 186.69 121.92))
-    (stroke (width 0) (type default))
-  )
-  (bus (pts (xy 88.9 100.33) (xy 99.06 100.33))
-    (stroke (width 0) (type default))
-  )
-  (bus (pts (xy 158.75 105.41) (xy 158.75 118.11))
-    (stroke (width 0) (type default))
-  )
-  (bus (pts (xy 111.76 120.65) (xy 111.76 125.73))
-    (stroke (width 0) (type default))
-  )
-  (bus (pts (xy 88.9 105.41) (xy 99.06 105.41))
-    (stroke (width 0) (type default))
-  )
-  (bus (pts (xy 111.76 125.73) (xy 111.76 128.27))
-    (stroke (width 0) (type default))
-  )
-  (bus (pts (xy 138.43 102.87) (xy 138.43 113.03))
-    (stroke (width 0) (type default))
-  )
-  (bus (pts (xy 162.56 102.87) (xy 162.56 90.17))
-    (stroke (width 0) (type default))
-  )
-  (bus (pts (xy 193.04 90.17) (xy 189.23 90.17))
-    (stroke (width 0) (type default))
-  )
-  (bus (pts (xy 182.88 113.03) (xy 193.04 113.03))
-    (stroke (width 0) (type default))
-  )
-  (bus (pts (xy 109.22 125.73) (xy 111.76 125.73))
-    (stroke (width 0) (type default))
-  )
-  (bus (pts (xy 193.04 92.71) (xy 186.69 92.71))
-    (stroke (width 0) (type default))
-  )
-  (bus (pts (xy 182.88 87.63) (xy 193.04 87.63))
-    (stroke (width 0) (type default))
-  )
-  (bus (pts (xy 148.59 73.66) (xy 148.59 76.2))
-    (stroke (width 0) (type default))
-  )
-  (bus (pts (xy 193.04 115.57) (xy 189.23 115.57))
-    (stroke (width 0) (type default))
-  )
-  (bus (pts (xy 162.56 83.82) (xy 162.56 90.17))
-    (stroke (width 0) (type default))
-  )
-  (bus (pts (xy 166.37 92.71) (xy 158.75 92.71))
-    (stroke (width 0) (type default))
-  )
-  (bus (pts (xy 162.56 115.57) (xy 162.56 102.87))
-    (stroke (width 0) (type default))
-  )
-  (bus (pts (xy 154.94 87.63) (xy 166.37 87.63))
-    (stroke (width 0) (type default))
-  )
-  (bus (pts (xy 158.75 118.11) (xy 166.37 118.11))
-    (stroke (width 0) (type default))
-  )
-  (bus (pts (xy 109.22 120.65) (xy 109.22 125.73))
-    (stroke (width 0) (type default))
-  )
   (label "S5" (at 182.88 113.03 180) (fields_autoplaced)
     (effects (font (size 1 1)) (justify right bottom))

Commit message: Nov 24th
Connections:
- net -5V: now also D1.2 (A), J1.1 (Pin_1), J2.2 (Pin_2), J3.2 (Pin_2), J4.2 (Pin_2), J5.2 (Pin_2), J6.2 (Pin_2), J7.2 (Pin_2)
- net GND: now also A1.29 (GND), A1.6 (GND), A1.7 (GND), J1.2 (Pin_2), J2.3 (Pin_3), J3.3 (Pin_3), J4.3 (Pin_3), J5.3 (Pin_3), J6.3 (Pin_3), J7.3 (Pin_3), R1.2
- net S0: now also A1.18 (D3), J2.1 (Pin_1)
- net S1: now also A1.20 (D5), J3.1 (Pin_1)
- net S2: now also A1.21 (D6), J4.1 (Pin_1)
- net S3: now also A1.24 (D9), J5.1 (Pin_1)
- net S4: now also A1.25 (D10), J6.1 (Pin_1)
- net S5: now also A1.26 (D11), J7.1 (Pin_1)
- net at D1.1 (K): now also R1.1
- no-connect marks 0 -> 22

Commit message: Dec25th
Parts:
- added J8: Conn_01x04, Connector_PinHeader_2.54mm:PinHeader_1x04_P2.54mm_Vertical, symbol Connector_Generic:Conn_01x04
Connections:
- net -5V: now also J8.3 (Pin_3)
- net GND: now also J8.4 (Pin_4)
- net SDA: now reaches A1.13 (SDA/A4)
- net SDA: now also J8.1 (Pin_1)
- net SCL: now reaches A1.14 (SCL/A5)
- net SCL: now also J8.2 (Pin_2)
- no-connect marks 22 -> 20
Changed lines of the file:
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@@
   (no_connect (at 95.25 97.79))
   (no_connect (at 95.25 95.25))
-  (no_connect (at 128.27 105.41))
   (no_connect (at 128.27 82.55))
   (no_connect (at 109.22 64.77))
@@
   (no_connect (at 128.27 77.47))
   (no_connect (at 128.27 95.25))
-  (no_connect (at 128.27 102.87))
   (no_connect (at 95.25 87.63))
   (no_connect (at 95.25 82.55))
@@
     (stroke (width 0) (type default))
   )
+  (wire (pts (xy 180.34 58.42) (xy 180.34 68.58))
+    (stroke (width 0) (type default))
+  )
   (wire (pts (xy 114.3 120.65) (xy 114.3 125.73))
     (stroke (width 0) (type default))
@@
     (stroke (width 0) (type default))
   )
+  (wire (pts (xy 180.34 68.58) (xy 193.04 68.58))
+    (stroke (width 0) (type default))
+  )
   (wire (pts (xy 138.43 72.39) (xy 138.43 81.28))
     (stroke (width 0) (type default))
@@
     (stroke (width 0) (type default))
   )
+  (wire (pts (xy 185.42 66.04) (xy 193.04 66.04))
+    (stroke (width 0) (type default))
+  )
   (wire (pts (xy 186.69 105.41) (xy 186.69 118.11))
     (stroke (width 0) (type default))
@@
     (stroke (width 0) (type default))
   )
+  (wire (pts (xy 185.42 71.12) (xy 185.42 72.39))
+    (stroke (width 0) (type default))
+  )
   (wire (pts (xy 189.23 115.57) (xy 193.04 115.57))
     (stroke (width 0) (type default))
@@
     (stroke (width 0) (type default))
   )
+  (wire (pts (xy 185.42 63.5) (xy 193.04 63.5))
+    (stroke (width 0) (type default))
+  )
   (wire (pts (xy 95.25 87.63) (xy 99.06 87.63))
     (stroke (width 0) (type default))
@@
     (stroke (width 0) (type default))
   )
+  (wire (pts (xy 124.46 102.87) (xy 128.27 102.87))
+    (stroke (width 0) (type default))
+  )
   (wire (pts (xy 162.56 102.87) (xy 162.56 115.57))
     (stroke (width 0) (type default))
@@
     (stroke (width 0) (type default))
   )
+  (wire (pts (xy 158.75 105.41) (xy 158.75 118.11))
+    (stroke (width 0) (type default))
+  )
+  (wire (pts (xy 189.23 102.87) (xy 193.04 102.87))
+    (stroke (width 0) (type default))
+  )
+  (wire (pts (xy 181.61 87.63) (xy 193.04 87.63))
+    (stroke (width 0) (type default))
+  )
+  (wire (pts (xy 193.04 71.12) (xy 185.42 71.12))
+    (stroke (width 0) (type default))
+  )
+  (wire (pts (xy 124.46 82.55) (xy 128.27 82.55))
+    (stroke (width 0) (type default))
+  )
+  (wire (pts (xy 95.25 82.55) (xy 99.06 82.55))
+    (stroke (width 0) (type default))
+  )
+  (wire (pts (xy 158.75 92.71) (xy 158.75 105.41))
+    (stroke (width 0) (type default))
+  )
   (wire (pts (xy 124.46 105.41) (xy 128.27 105.41))
     (stroke (width 0) (type default))
   )
-  (wire (pts (xy 158.75 105.41) (xy 158.75 118.11))
-    (stroke (width 0) (type default))
-  )
-  (wire (pts (xy 189.23 102.87) (xy 193.04 102.87))
-    (stroke (width 0) (type default))
-  )
-  (wire (pts (xy 124.46 102.87) (xy 128.27 102.87))
-    (stroke (width 0) (type default))
-  )
-  (wire (pts (xy 181.61 87.63) (xy 193.04 87.63))
-    (stroke (width 0) (type default))
-  )
-  (wire (pts (xy 124.46 82.55) (xy 128.27 82.55))
-    (stroke (width 0) (type default))
-  )
-  (wire (pts (xy 95.25 82.55) (xy 99.06 82.55))
-    (stroke (width 0) (type default))
-  )
-  (wire (pts (xy 158.75 92.71) (xy 158.75 105.41))
-    (stroke (width 0) (type default))
+  (label "SCL" (at 185.42 66.04 0) (fields_autoplaced)
+    (effects (font (size 1.27 1.27)) (justify left bottom))
   )
   (label "S0" (at 86.36 85.09 0) (fields_autoplaced)
     (effects (font (size 1 1)) (justify left bottom))
   )
+  (label "SDA" (at 185.42 63.5 0) (fields_autoplaced)
+    (effects (font (size 1.27 1.27)) (justify left bottom))
+  )
   (label "S2" (at 153.67 113.03 0) (fields_autoplaced)
     (effects (font (size 1 1)) (justify left bottom))
   )
+  (label "SCL" (at 128.27 105.41 0) (fields_autoplaced)
+    (effects (font (size 1.27 1.27)) (justify left bottom))
+  )
   (label "S1" (at 153.67 100.33 0) (fields_autoplaced)
     (effects (font (size 1 1)) (justify left bottom))
+  )
+  (label "SDA" (at 128.27 102.87 0) (fields_autoplaced)
+    (effects (font (size 1.27 1.27)) (justify left bottom))
   )
   (label "S4" (at 86.36 102.87 0) (fields_autoplaced)
@@
       (effects (font (size 1.27 1.27)) hide)
     )
-    (pin "32")
-    (pin "21")
-    (pin "27")
-    (pin "7")
+    (pin "1")
+    (pin "10")
+    (pin "11")
+    (pin "12")
+    (pin "13")
+    (pin "14")
+    (pin "15")
+    (pin "16")
+    (pin "17")
     (pin "18")
     (pin "19")
-    (pin "4")
-    (pin "10")
+    (pin "2")
+    (pin "20")
+    (pin "21")
     (pin "22")
-    (pin "11")
-    (pin "6")
     (pin "23")
-    (pin "28")
-    (pin "15")
-    (pin "17")
     (pin "24")
     (pin "25")
-    (pin "14")
-    (pin "12")
-    (pin "20")
-    (pin "8")
+    (pin "26")
+    (pin "27")
+    (pin "28")
+    (pin "29")
     (pin "3")
     (pin "30")
+    (pin "31")
+    (pin "32")
+    (pin "4")
     (pin "5")
-    (pin "13")
-    (pin "29")
+    (pin "6")
+    (pin "7")
+    (pin "8")
     (pin "9")
-    (pin "1")
-    (pin "26")
-    (pin "31")
-    (pin "2")
-    (pin "16")
     (instances
       (project "arduino_robotarm_shield"
@@
       (effects (font (size 1.27 1.27)) hide)
     )
-    (pin "2")
-    (pin "1")
+    (pin "1")
+    (pin "2")
     (pin "3")
     (instances
@@
       (effects (font (size 1.27 1.27)) hide)
     )
-    (pin "2")
-    (pin "1")
+    (pin "1")
+    (pin "2")
     (pin "3")
     (instances
@@
       (effects (font (size 1.27 1.27)) hide)
     )
-    (pin "2")
-    (pin "1")
+    (pin "1")
+    (pin "2")
     (instances
       (project "arduino_robotarm_shield"
@@
     )
   )
+  (symbol (lib_id "power:-5V") (at 180.34 58.42 0) (unit 1)
+    (in_bom yes) (on_board yes) (dnp no) (fields_autoplaced)
+    (property "Reference" "#PWR011" (at 180.34 55.88 0)
+      (effects (font (size 1.27 1.27)) hide)
+    )
+    (property "Value" "-5V" (at 180.34 53.34 0)
+      (effects (font (size 1.27 1.27)))
+    )
+    (property "Footprint" "" (at 180.34 58.42 0)
+      (effects (font (size 1.27 1.27)) hide)
+    )
+    (property "Datasheet" "" (at 180.34 58.42 0)
+      (effects (font (size 1.27 1.27)) hide)
+    )
+    (pin "1")
+    (instances
+      (project "arduino_robotarm_shield"
+        (path "/5a003089-c902-4e4a-9db6-c278bc971473"
+          (reference "#PWR011") (unit 1)
+        )
+      )
+    )
+  )
   (symbol (lib_id "Connector_Generic:Conn_01x03") (at 198.12 115.57 0) (unit 1)
     (in_bom yes) (on_board yes) (dnp no) (fields_autoplaced)
@@
       (effects (font (size 1.27 1.27)) hide)
     )
-    (pin "2")
-    (pin "1")
+    (pin "1")
+    (pin "2")
     (pin "3")
     (instances
@@
       (effects (font (size 1.27 1.27)) hide)
     )
-    (pin "2")
-    (pin "1")
+    (pin "1")
+    (pin "2")
     (pin "3")
     (instances
@@
       (effects (font (size 1.27 1.27)) hide)
     )
-    (pin "2")
-    (pin "1")
+    (pin "1")
+    (pin "2")
     (pin "3")
     (instances
@@
       (effects (font (size 1.27 1.27)) hide)
     )
-    (pin "2")
-    (pin "1")
+    (pin "1")
+    (pin "2")
     (pin "3")
     (instances
@@
         )
       )
+    )
+  )
+  (symbol (lib_id "power:GND") (at 185.42 72.39 0) (unit 1)
+    (in_bom yes) (on_board yes) (dnp no)
+    (property "Reference" "#PWR012" (at 185.42 78.74 0)
+      (effects (font (size 1.27 1.27)) hide)
+    )
+    (property "Value" "GND" (at 185.42 76.2 0)
+      (effects (font (size 1.27 1.27)))
+    )
+    (property "Footprint" "" (at 185.42 72.39 0)
+      (effects (font (size 1.27 1.27)) hide)
+    )
+    (property "Datasheet" "" (at 185.42 72.39 0)
+      (effects (font (size 1.27 1.27)) hide)
+    )
+    (pin "1")
+    (instances
+      (project "arduino_robotarm_shield"
+        (path "/5a003089-c902-4e4a-9db6-c278bc971473"
+          (reference "#PWR012") (unit 1)
+        )
+      )
+    )
+  )
+  (symbol (lib_id "Connector_Generic:Conn_01x04") (at 198.12 66.04 0) (unit 1)
+    (in_bom yes) (on_board yes) (dnp no) (fields_autoplaced)
+    (property "Reference" "J8" (at 200.66 66.04 0)
+      (effects (font (size 1.27 1.27)) (justify left))
+    )
+    (property "Value" "Conn_01x04" (at 200.66 68.58 0)
+      (effects (font (size 1.27 1.27)) (justify left))
+    )
+    (property "Footprint" "Connector_PinHeader_2.54mm:PinHeader_1x04_P2.54mm_Vertical" (at 198.12 66.04 0)
+      (effects (font (size 1.27 1.27)) hide)
+    )
+    (property "Datasheet" "~" (at 198.12 66.04 0)
+      (effects (font (size 1.27 1.27)) hide)
+    )
+    (pin "1")
+    (pin "2")
+    (pin "3")
+    (pin "4")
+    (instances
+      (project "arduino_robotarm_shield"
+        (path "/5a003089-c902-4e4a-9db6-c278bc971473"
+          (reference "J8") (unit 1)
+        )
+      )
